File: LedLights/kicad/led-lights.sch (KiCad schematic (older format))
At the start: 6 parts, among them CON1 BARREL_JACK, P1 LDR connector, P2 PIR connector, P3 LED driver conn, U1 arduino_nano

Commit message: KiCad stuff, schema, and pcb
Parts:
- removed CON1: BARREL_JACK, symbol BARREL_JACK
- removed P3: LED driver conn, symbol CONN_01X03
- added P1: Power input, Connect:AK300-2, symbol CONN_01X02
- added P4: Power output, Connect:AK300-2, symbol CONN_01X02
- added P5: LED 1, Connect:AK300-2, symbol CONN_01X02
- added P6: LED 2, Connect:AK300-2, symbol CONN_01X02
- added P7: PIR2 connector, Connect:AK300-4, symbol CONN_01X04
- added P8: LED 3, Connect:AK300-2, symbol CONN_01X02
- P2: value PIR connector -> PIR1 connector; footprint (none) -> Connect:AK300-4; symbol CONN_01X03 -> CONN_01X04
- P3: renamed from P1; footprint (none) -> Connect:AK300-2
- R1: footprint (none) -> Resistors_ThroughHole:Resistor_Horizontal_RM15mm; symbol R -> R-RESCUE-led-lights
- U1: footprint DIL20 -> lib:arduino_nano
Connections:
- net +12V: now also P1.1 (P1), P4.1 (P1); no longer P2.1 (P1)
- net +5V: now also P2.1 (P1), P7.1 (P1)
- net GND: now also P5.2 (P2), P6.2 (P2), P7.3 (P3), P8.2 (P2)
- net ledPwmPin1: now reaches U1.D3 (#D3)
- net ledPwmPin1: now also P5.1 (P1)
- net pirInPin2: now reaches U1.D4
- net pirInPin2: now also P7.2 (P2)
- net ledPwmPin2: now reaches U1.D5 (#D5)
- net ledPwmPin2: now also P6.1 (P1)
- net ledPwmPin3: now reaches U1.D6 (#D6)
- net ledPwmPin3: now also P8.1 (P1)
- net LedLightPwm: no longer names the net of U1.D9 (#D9)
- net MotionSensor renamed pirInPin1
- new net GNDPWR: P1.2 (P2), P4.2 (P2)
- no-connect marks 15 -> 22

Commit message: KiCad + program change.
Parts:
- removed P4: Power output, Connect:AK300-2, symbol CONN_01X02
Connections:
- net GNDPWR is gone; now on net GND: P1.2 (P2)
Changed lines of the file:
@@
 NoConn ~ 10150 1450
-$Comp
-L CONN_01X02 P4
-U 1 1 55FFD153
-P 10350 2900
-F 0 "P4" H 10350 3050 50  0000 C CNN
-F 1 "Power output" V 10450 2900 50  0000 C CNN
-F 2 "Connect:AK300-2" H 10350 2900 60  0001 C CNN
-F 3 "" H 10350 2900 60  0000 C CNN
-	1    10350 2900
-	1    0    0    -1
-$EndComp
-Wire Wire Line
-	9900 2850 10150 2850
-Wire Wire Line
-	9900 3050 9900 2950
-Wire Wire Line
-	9900 2950 10150 2950
 $Comp
 L CONN_01X02 P5
@@
 NoConn ~ 4550 3900
 $Comp
-L +12V #PWR015
-U 1 1 56001582
-P 9900 2850
-F 0 "#PWR015" H 9900 2700 50  0001 C CNN
-F 1 "+12V" H 9900 2990 50  0000 C CNN
-F 2 "" H 9900 2850 60  0000 C CNN
-F 3 "" H 9900 2850 60  0000 C CNN
-	1    9900 2850
-	0    -1   -1   0
-$EndComp
-$Comp
-L GNDPWR #PWR016
-U 1 1 55FFE777
+L GND #PWR?
+U 1 1 560286AB
 P 2250 2500
-F 0 "#PWR016" H 2250 2300 50  0001 C CNN
-F 1 "GNDPWR" H 2250 2370 50  0000 C CNN
-F 2 "" H 2250 2450 60  0000 C CNN
-F 3 "" H 2250 2450 60  0000 C CNN
+F 0 "#PWR?" H 2250 2250 50  0001 C CNN
+F 1 "GND" H 2250 2350 50  0000 C CNN
+F 2 "" H 2250 2500 60  0000 C CNN
+F 3 "" H 2250 2500 60  0000 C CNN
 	1    2250 2500
 	1    0    0    -1
 $EndComp
 Wire Wire Line
-	2250 2500 2250 2300
+	1850 2300 2250 2300
 Wire Wire Line
-	2250 2300 1850 2300
-$Comp
-L GNDPWR #PWR017
-U 1 1 55FFEEDC
-P 9900 3050
-F 0 "#PWR017" H 9900 2850 50  0001 C CNN
-F 1 "GNDPWR" H 9900 2920 50  0000 C CNN
-F 2 "" H 9900 3000 60  0000 C CNN
-F 3 "" H 9900 3000 60  0000 C CNN
-	1    9900 3050
-	1    0    0    -1
-$EndComp
+	2250 2300 2250 2500
 $EndSCHEMATC
