File: LedLights/kicad/led-lights.sch (KiCad schematic (older format))
At the start: 9 parts, among them P1 Power input, P2 PIR1 connector, P3 LDR connector, P5 LED 1, P6 LED 2, P7 PIR2 connector, P8 LED 3, U1 arduino_nano

Commit message: Kicad
Parts:
- added P9: HC-05 connector, Socket_Strips:Socket_Strip_Straight_1x04, symbol CONN_01X04
Connections:
- net +5V: now also P9.1 (P1)
- net GND: now also P9.2 (P2)
- net RX: now reaches U1.RX0
- net RX: now also P9.3 (P3)
- net TX: now reaches U1.TX1
- net TX: now also P9.4 (P4)
- no-connect marks 22 -> 20
Changed lines of the file:
@@
 NoConn ~ 3150 4400
 NoConn ~ 3150 4600
-NoConn ~ 4550 4800
-NoConn ~ 4550 4700
 NoConn ~ 4550 4600
 Wire Wire Line
@@
 NoConn ~ 4550 3900
 $Comp
-L GND #PWR?
+L GND #PWR015
 U 1 1 560286AB
 P 2250 2500
-F 0 "#PWR?" H 2250 2250 50  0001 C CNN
+F 0 "#PWR015" H 2250 2250 50  0001 C CNN
 F 1 "GND" H 2250 2350 50  0000 C CNN
 F 2 "" H 2250 2500 60  0000 C CNN
@@
 Wire Wire Line
 	2250 2300 2250 2500
+$Comp
+L CONN_01X04 P9
+U 1 1 561E4F57
+P 10350 2950
+F 0 "P9" H 10350 3186 50  0000 C CNN
+F 1 "HC-05 connector" V 10450 2950 50  0000 C CNN
+F 2 "Socket_Strips:Socket_Strip_Straight_1x04" H 10350 2950 60  0001 C CNN
+F 3 "" H 10350 2950 60  0000 C CNN
+	1    10350 2950
+	1    0    0    -1
+$EndComp
+$Comp
+L +5V #PWR016
+U 1 1 561E5B3C
+P 9750 2800
+F 0 "#PWR016" H 9750 2650 50  0001 C CNN
+F 1 "+5V" H 9750 2940 50  0000 C CNN
+F 2 "" H 9750 2800 60  0000 C CNN
+F 3 "" H 9750 2800 60  0000 C CNN
+	1    9750 2800
+	0    -1   -1   0
+$EndComp
+Wire Wire Line
+	9750 2800 10150 2800
+$Comp
+L GND #PWR017
+U 1 1 561E7145
+P 9350 2900
+F 0 "#PWR017" H 9350 2650 50  0001 C CNN
+F 1 "GND" H 9350 2750 50  0000 C CNN
+F 2 "" H 9350 2900 60  0000 C CNN
+F 3 "" H 9350 2900 60  0000 C CNN
+	1    9350 2900
+	0    1    1    0
+$EndComp
+Wire Wire Line
+	10150 2900 9350 2900
+Text GLabel 10000 3000 0    60   Output ~ 0
+RX
+Wire Wire Line
+	10150 3000 10000 3000
+Text GLabel 9750 3100 0    60   Input ~ 0
+TX
+Wire Wire Line
+	10150 3100 9750 3100
+Text GLabel 5100 4700 2    60   Input ~ 0
+RX
+Wire Wire Line
+	5100 4700 4550 4700
+Text GLabel 4900 4800 2    60   Output ~ 0
+TX
+Wire Wire Line
+	4550 4800 4900 4800
 $EndSCHEMATC
