File: LedLights/kicad/led-lights.kicad_pcb (KiCad board)
At the start: 2 copper layers, 10 parts, among them P1 Power input, P2 PIR1 connector, P3 LDR connector, P4 Power output, P5 LED 1, P6 LED 2, P7 PIR2 connector, P8 LED 3, U1 arduino_nano

Commit message: KiCad + program change.
Parts:
- removed P4: Power output, Connect:AK300-2
- moved P8 32.5 mm to (67.3, 54.6), turned to 270 degrees
- moved R1 32.4 mm to (53.3, 21.6)
- moved P6 28.7 mm to (67.3, 41.9), turned to 270 degrees
- moved P5 25.4 mm to (67.3, 29.2), turned to 270 degrees
- moved P2 16.5 mm to (17.8, 66.0), turned to 0 degrees
- moved P7 16.5 mm to (40.6, 66.0), turned to 0 degrees
- moved P3 12.7 mm to (30.5, 20.3)
Connections:
- P1 pad 2: GNDPWR -> GND
- P2 pad 4: Net-(P2-Pad4) -> (no net)
- P7 pad 4: Net-(P7-Pad4) -> (no net)
- U1 pad 3V3: Net-(U1-Pad3V3) -> (no net)
- U1 pad A1: Net-(U1-PadA1) -> (no net)
- U1 pad A2: Net-(U1-PadA2) -> (no net)
- U1 pad A3: Net-(U1-PadA3) -> (no net)
- U1 pad A4: Net-(U1-PadA4) -> (no net)
- U1 pad A5: Net-(U1-PadA5) -> (no net)
- U1 pad A6: Net-(U1-PadA6) -> (no net)
- U1 pad A7: Net-(U1-PadA7) -> (no net)
- U1 pad D10: Net-(U1-PadD10) -> (no net)
- U1 pad D11: Net-(U1-PadD11) -> (no net)
- U1 pad D12: Net-(U1-PadD12) -> (no net)
- U1 pad D13: Net-(U1-PadD13) -> (no net)
- U1 pad D7: Net-(U1-PadD7) -> (no net)
- U1 pad D8: Net-(U1-PadD8) -> (no net)
- U1 pad D9: Net-(U1-PadD9) -> (no net)
- U1 pad REF: Net-(U1-PadREF) -> (no net)
- U1 pad RST: Net-(U1-PadRST) -> (no net)
- U1 pad RX0: Net-(U1-PadRX0) -> (no net)
- U1 pad TX1: Net-(U1-PadTX1) -> (no net)
Routing:
- net GND: track 0.00 -> 231.8 mm
- net +5V: track 0.00 -> 92.2 mm, vias 0 -> 2
- net ledPwmPin1: track 0.00 -> 56.0 mm
- net ledPwmPin3: track 0.00 -> 40.7 mm
- net ledPwmPin2: track 0.00 -> 39.7 mm
- net Net-(P3-Pad2): track 0.00 -> 26.2 mm
- net pirInPin2: track 0.00 -> 24.5 mm
- net +12V: track 0.00 -> 16.5 mm
- net pirInPin1: track 0.00 -> 16.1 mm
Other:
- net class 12V added: clearance 0.5, trace_width 1.5, via_dia 2.5, via_drill 0.75
- net class Default: clearance 0.2 -> 0.254; trace_width 0.25 -> 1; via_dia 0.6 -> 2; via_drill 0.4 -> 0.75
- net class GND added: clearance 0.5, trace_width 1.5, via_dia 2.5, via_drill 0.75
- rule trace_clearance: 0.2 -> 0.254

Commit message: kicad
Parts:
- moved P3 113.0 mm to (132.1, 69.8)
- moved P7 113.0 mm to (142.2, 115.6)
- moved U1 113.0 mm to (138.4, 94.0)
- moved P1 113.0 mm to (119.4, 69.8)
- moved P2 113.0 mm to (119.4, 115.6)
- moved P5 113.0 mm to (168.9, 78.7)
- moved P6 113.0 mm to (168.9, 91.4)
- moved P8 113.0 mm to (168.9, 104.1)
- moved R1 113.0 mm to (154.9, 71.1)
Routing:
- net GND: track 231.8 -> 255.6 mm
Other:
- board outline added: 71.1 x 71.1 mm
