File: LedLights/kicad/led-lights.kicad_pcb (KiCad board)
At the start: 2 copper layers, 71.1 x 71.1 mm, 9 parts, among them P1 Power input, P2 PIR1 connector, P3 LDR connector, P5 LED 1, P6 LED 2, P7 PIR2 connector, P8 LED 3, U1 arduino_nano

Commit message: Kicad
Parts:
- added REF**: 1pin, Connect:1pin, F.Cu at (180.3, 62.2)
- added REF**: 1pin, Connect:1pin, F.Cu at (180.3, 125.7)
- added REF**: 1pin, Connect:1pin, F.Cu at (116.0, 81.3)
- added REF**: 1pin, Connect:1pin, F.Cu at (116.8, 125.7)
- added REF**: 1pin, Connect:1pin, F.Cu at (143.5, 67.3)
Changed lines of the file:
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@@
     (links 18)
     (no_connects 0)
-    (area 113.029499 58.369999 184.200001 129.590001)
+    (area 113.029499 57.757 184.200001 129.799)
     (thickness 1.6)
-    (drawings 5)
+    (drawings 8)
     (tracks 81)
     (zones 0)
-    (modules 9)
+    (modules 14)
     (nets 10)
   )
@@
       (subtractmaskfromsilk false)
       (outputformat 4)
-      (mirror true)
+      (mirror false)
       (drillshape 1)
       (scaleselection 1)
@@
       (net 1 +12V))
   )
+  (module Connect:1pin (layer F.Cu)
+    (at 180.34 62.23)
+    (descr "module 1 pin (ou trou mecanique de percage)")
+    (tags DEV)
+    (fp_text reference REF** (at 0 -3.048) (layer F.SilkS)
+      (effects (font (size 1 1) (thickness 0.15)))
+    )
+    (fp_text value 1pin (at 0 2.794) (layer F.Fab)
+      (effects (font (size 1 1) (thickness 0.15)))
+    )
+    (fp_circle (center 0 0) (end 0 -2.286) (layer F.SilkS) (width 0.15))
+    (pad 1 thru_hole circle (at 0 0) (size 4.064 4.064) (drill 3.048) (layers *.Cu *.Mask F.SilkS))
+  )
+  (module Connect:1pin (layer F.Cu)
+    (at 180.34 125.73)
+    (descr "module 1 pin (ou trou mecanique de percage)")
+    (tags DEV)
+    (fp_text reference REF** (at 0 -3.048) (layer F.SilkS)
+      (effects (font (size 1 1) (thickness 0.15)))
+    )
+    (fp_text value 1pin (at 0 2.794) (layer F.Fab)
+      (effects (font (size 1 1) (thickness 0.15)))
+    )
+    (fp_circle (center 0 0) (end 0 -2.286) (layer F.SilkS) (width 0.15))
+    (pad 1 thru_hole circle (at 0 0) (size 4.064 4.064) (drill 3.048) (layers *.Cu *.Mask F.SilkS))
+  )
+  (module Connect:1pin (layer F.Cu)
+    (at 116 81.28)
+    (descr "module 1 pin (ou trou mecanique de percage)")
+    (tags DEV)
+    (fp_text reference REF** (at 0 -3.048) (layer F.SilkS)
+      (effects (font (size 1 1) (thickness 0.15)))
+    )
+    (fp_text value 1pin (at 0 2.794) (layer F.Fab)
+      (effects (font (size 1 1) (thickness 0.15)))
+    )
+    (fp_circle (center 0 0) (end 0 -2.286) (layer F.SilkS) (width 0.15))
+    (pad 1 thru_hole circle (at 0 0) (size 4.064 4.064) (drill 3.048) (layers *.Cu *.Mask F.SilkS))
+  )
+  (module Connect:1pin (layer F.Cu)
+    (at 116.84 125.73)
+    (descr "module 1 pin (ou trou mecanique de percage)")
+    (tags DEV)
+    (fp_text reference REF** (at 0 -3.048) (layer F.SilkS)
+      (effects (font (size 1 1) (thickness 0.15)))
+    )
+    (fp_text value 1pin (at 0 2.794) (layer F.Fab)
+      (effects (font (size 1 1) (thickness 0.15)))
+    )
+    (fp_circle (center 0 0) (end 0 -2.286) (layer F.SilkS) (width 0.15))
+    (pad 1 thru_hole circle (at 0 0) (size 4.064 4.064) (drill 3.048) (layers *.Cu *.Mask F.SilkS))
+  )
+  (module Connect:1pin (layer F.Cu)
+    (at 143.51 67.31)
+    (descr "module 1 pin (ou trou mecanique de percage)")
+    (tags DEV)
+    (fp_text reference REF** (at 0 -3.048) (layer F.SilkS)
+      (effects (font (size 1 1) (thickness 0.15)))
+    )
+    (fp_text value 1pin (at 0 2.794) (layer F.Fab)
+      (effects (font (size 1 1) (thickness 0.15)))
+    )
+    (fp_circle (center 0 0) (end 0 -2.286) (layer F.SilkS) (width 0.15))
+    (pad 1 thru_hole circle (at 0 0) (size 4.064 4.064) (drill 3.048) (layers *.Cu *.Mask F.SilkS))
+  )
+  (dimension 71.12 (width 0.3) (layer Dwgs.User)
+    (gr_text "71,120 mm" (at 148.59 139.78) (layer Dwgs.User)
+      (effects (font (size 1.5 1.5) (thickness 0.3)))
+    )
+    (feature1 (pts (xy 184.15 129.54) (xy 184.15 141.13)))
+    (feature2 (pts (xy 113.03 129.54) (xy 113.03 141.13)))
+    (crossbar (pts (xy 113.03 138.43) (xy 184.15 138.43)))
+    (arrow1a (pts (xy 184.15 138.43) (xy 183.023496 139.016421)))
+    (arrow1b (pts (xy 184.15 138.43) (xy 183.023496 137.843579)))
+    (arrow2a (pts (xy 113.03 138.43) (xy 114.156504 139.016421)))
+    (arrow2b (pts (xy 113.03 138.43) (xy 114.156504 137.843579)))
+  )
+  (dimension 63.5 (width 0.3) (layer Dwgs.User)
+    (gr_text "63,500 mm" (at 148.59 134.7) (layer Dwgs.User)
+      (effects (font (size 1.5 1.5) (thickness 0.3)))
+    )
+    (feature1 (pts (xy 180.34 125.73) (xy 180.34 136.05)))
+    (feature2 (pts (xy 116.84 125.73) (xy 116.84 136.05)))
+    (crossbar (pts (xy 116.84 133.35) (xy 180.34 133.35)))
+    (arrow1a (pts (xy 180.34 133.35) (xy 179.213496 133.936421)))
+    (arrow1b (pts (xy 180.34 133.35) (xy 179.213496 132.763579)))
+    (arrow2a (pts (xy 116.84 133.35) (xy 117.966504 133.936421)))
+    (arrow2b (pts (xy 116.84 133.35) (xy 117.966504 132.763579)))
+  )
+  (dimension 71.12 (width 0.3) (layer Dwgs.User)
+    (gr_text "71,120 mm" (at 190.58 93.98 270) (layer Dwgs.User)
+      (effects (font (size 1.5 1.5) (thickness 0.3)))
+    )
+    (feature1 (pts (xy 184.15 129.54) (xy 191.93 129.54)))
+    (feature2 (pts (xy 184.15 58.42) (xy 191.93 58.42)))
+    (crossbar (pts (xy 189.23 58.42) (xy 189.23 129.54)))
+    (arrow1a (pts (xy 189.23 129.54) (xy 188.643579 128.413496)))
+    (arrow1b (pts (xy 189.23 129.54) (xy 189.816421 128.413496)))
+    (arrow2a (pts (xy 189.23 58.42) (xy 188.643579 59.546504)))
+    (arrow2b (pts (xy 189.23 58.42) (xy 189.816421 59.546504)))
+  )
   (gr_line (start 184.15 58.42) (end 184.15 129.54) (angle 90) (layer Edge.Cuts) (width 0.001))
