File: LedLights/kicad/led-lights.kicad_pcb (KiCad board)
At the start: 2 copper layers, 71.1 x 71.1 mm, 14 parts, among them P1 Power input, P2 PIR1 connector, P3 LDR connector, P5 LED 1, P6 LED 2, P7 PIR2 connector, P8 LED 3, U1 arduino_nano

Commit message: Kicad
Parts:
- added P9: HC-05 connector, Socket_Strips:Socket_Strip_Straight_1x04, F.Cu at (108.0, 91.4)
- moved REF** 21.8 mm to (105.4, 62.2)
- moved REF** 11.4 mm to (105.4, 125.7)
Connections:
- U1 pad RX0: (no net) -> RX
- U1 pad TX1: (no net) -> TX
Routing:
- net +5V: track 92.2 -> 118.5 mm, vias 2 -> 4
- net GND: track 255.6 -> 275.7 mm
- net RX: track 0.00 -> 18.3 mm
- net TX: track 0.00 -> 12.5 mm
Other:
- board size 71.1 x 71.1 mm -> 82.6 x 71.1 mm
