File: LedLights/kicad/v0.2/led-lights.sch (KiCad schematic (older format))
At the start: 10 parts, among them P1 Power input, P2 PIR1 connector, P3 LDR connector, P5 LED 1, P6 LED 2, P7 PIR2 connector, P8 LED 3, P9 HC-05 connector, U1 arduino_nano

Commit message: Kicad and stuff
Parts:
- added U2, U3, U4: LED_Driver_700mA, lib:LED_Driver_700mA_foot, symbol LED_Driver_700mA
- P1: footprint Connect:AK300-2 -> Connectors:AK300-2
- P2: renamed from P3; footprint Connect:AK300-2 -> Connectors:AK300-2
- P3: renamed from P5; footprint Connect:AK300-2 -> Connectors:AK300-2
- P4: renamed from P6; footprint Connect:AK300-2 -> Connectors:AK300-2
- P5: renamed from P8; footprint Connect:AK300-2 -> Connectors:AK300-2
- P6: renamed from P2; footprint Connect:AK300-4 -> Connectors:AK300-4
- P7: footprint Connect:AK300-4 -> Connectors:AK300-4
- P8: renamed from P9; footprint Socket_Strips:Socket_Strip_Straight_1x04 -> Socket_Strips:Socket_Strip_Straight_1x04_Pitch2.54mm
- R1: footprint Resistors_ThroughHole:Resistor_Horizontal_RM15mm -> Resistors_General:Resistor_Horizontal_RM15mm
Connections:
- net +12V: now also U2.1 (VIN+), U3.1 (VIN+), U4.1 (VIN+)
- net GND: now also U2.2 (VIN-), U2.6 (GND), U3.2 (VIN-), U3.6 (GND), U4.2 (VIN-), U4.6 (GND); no longer P3.2 (P2), P4.2 (P2), P5.2 (P2)
- net ledPwmPin1: now also U2.5 (PWM); no longer P3.1 (P1)
- net ledPwmPin2: now also U3.5 (PWM); no longer P4.1 (P1)
- net ledPwmPin3: now also U4.5 (PWM); no longer P5.1 (P1)
- new net: P3.1 (P1), U2.3 (LED+)
- new net: P3.2 (P2), U2.4 (LED-)
- new net: P4.1 (P1), U3.3 (LED+)
- new net: P4.2 (P2), U3.4 (LED-)
- new net: P5.1 (P1), U4.3 (LED+)
- new net: P5.2 (P2), U4.4 (LED-)
Other:
- moved on the sheet: P3, P4, P5
